File: mm_external_uart.kicad_sch (KiCad schematic)
At the start: 0 parts

Commit message: fin tp2
Parts:
- added C13: 2.2uF, Capacitor_SMD:C_0603_1608Metric, symbol minimouse:C
- added C17: 0.1uF, Capacitor_SMD:C_0603_1608Metric, symbol minimouse:C
- added J4: Conn_01x04, Connector_PinHeader_2.54mm:PinHeader_1x04_P2.54mm_Vertical, symbol Connector_Generic:Conn_01x04
- added R19: 100, Resistor_SMD:R_0603_1608Metric, symbol minimouse:R
Connections:
- new net: J4.3 (Pin_3), R19.2
- new net +BATT: C13.1, C17.1, J4.1 (Pin_1)
- new net EXT_UART_RX: J4.4 (Pin_4)
- new net EXT_UART_TX: R19.1
- new net GND: C13.2, C17.2, J4.2 (Pin_2)
Changed lines of the file:
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@@
 (kicad_sch (version 20230121) (generator eeschema)
   (paper "A4")
+  (junction (at 123.19 73.66) (diameter 0) (color 0 0 0 0)
+  )
+  (junction (at 123.19 81.28) (diameter 0) (color 0 0 0 0)
+  )
+  (wire (pts (xy 123.19 81.28) (xy 123.19 85.09))
+    (stroke (width 0) (type default))
+  )
+  (wire (pts (xy 149.86 90.17) (xy 151.13 90.17))
+    (stroke (width 0) (type default))
+  )
+  (wire (pts (xy 149.86 92.71) (xy 160.02 92.71))
+    (stroke (width 0) (type default))
+  )
+  (wire (pts (xy 151.13 85.09) (xy 160.02 85.09))
+    (stroke (width 0) (type default))
+  )
+  (wire (pts (xy 158.75 90.17) (xy 160.02 90.17))
+    (stroke (width 0) (type default))
+  )
+  (wire (pts (xy 123.19 69.85) (xy 123.19 73.66))
+    (stroke (width 0) (type default))
+  )
+  (wire (pts (xy 110.49 81.28) (xy 123.19 81.28))
+    (stroke (width 0) (type default))
+  )
+  (wire (pts (xy 130.81 97.79) (xy 130.81 87.63))
+    (stroke (width 0) (type default))
+  )
+  (wire (pts (xy 151.13 80.01) (xy 151.13 85.09))
+    (stroke (width 0) (type default))
+  )
+  (wire (pts (xy 130.81 87.63) (xy 160.02 87.63))
+    (stroke (width 0) (type default))
+  )
+  (wire (pts (xy 110.49 73.66) (xy 123.19 73.66))
+    (stroke (width 0) (type default))
+  )
+  (hierarchical_label "EXT_UART_RX" (shape input) (at 149.86 92.71 180) (fields_autoplaced)
+    (effects (font (size 1.27 1.27)) (justify right))
+  )
+  (hierarchical_label "EXT_UART_TX" (shape output) (at 149.86 90.17 180) (fields_autoplaced)
+    (effects (font (size 1.27 1.27)) (justify right))
+  )
+  (symbol (lib_id "minimouse:C") (at 110.49 77.47 0) (unit 1)
+    (in_bom yes) (on_board yes) (dnp no) (fields_autoplaced)
+    (property "Reference" "C17" (at 114.3 76.2 0)
+      (effects (font (size 1.27 1.27)) (justify left) hide)
+    )
+    (property "Value" "0.1uF" (at 114.3 78.74 0)
+      (effects (font (size 1.27 1.27)) (justify left))
+    )
+    (property "Footprint" "Capacitor_SMD:C_0603_1608Metric" (at 111.4552 81.28 0)
+      (effects (font (size 1.27 1.27)) hide)
+    )
+    (property "Datasheet" "~" (at 110.49 77.47 0)
+      (effects (font (size 1.27 1.27)) hide)
+    )
+    (pin "1")
+    (pin "2")
+    (instances
+      (project "minimouse"
+        (path "/d8fa4cba-2469-4231-847f-065b6b829f44/224298a9-7d6e-4a70-a0a5-f2614895ec28"
+          (reference "C17") (unit 1)
+        )
+        (path "/d8fa4cba-2469-4231-847f-065b6b829f44/d17bb1c7-f68a-465e-9a17-5858ef86fc30"
+          (reference "C18") (unit 1)
+        )
+      )
+    )
+  )
+  (symbol (lib_id "minimouse:C") (at 123.19 77.47 0) (unit 1)
+    (in_bom yes) (on_board yes) (dnp no) (fields_autoplaced)
+    (property "Reference" "C13" (at 127 76.2 0)
+      (effects (font (size 1.27 1.27)) (justify left) hide)
+    )
+    (property "Value" "2.2uF" (at 127 78.74 0)
+      (effects (font (size 1.27 1.27)) (justify left))
+    )
+    (property "Footprint" "Capacitor_SMD:C_0603_1608Metric" (at 124.1552 81.28 0)
+      (effects (font (size 1.27 1.27)) hide)
+    )
+    (property "Datasheet" "~" (at 123.19 77.47 0)
+      (effects (font (size 1.27 1.27)) hide)
+    )
+    (pin "1")
+    (pin "2")
+    (instances
+      (project "minimouse"
+        (path "/d8fa4cba-2469-4231-847f-065b6b829f44/d17bb1c7-f68a-465e-9a17-5858ef86fc30"
+          (reference "C13") (unit 1)
+        )
+      )
+    )
+  )
+  (symbol (lib_id "power:+BATT") (at 151.13 80.01 0) (unit 1)
+    (in_bom yes) (on_board yes) (dnp no) (fields_autoplaced)
+    (property "Reference" "#PWR023" (at 151.13 83.82 0)
+      (effects (font (size 1.27 1.27)) hide)
+    )
+    (property "Value" "+BATT" (at 151.13 74.93 0)
+      (effects (font (size 1.27 1.27)))
+    )
+    (property "Footprint" "" (at 151.13 80.01 0)
+      (effects (font (size 1.27 1.27)) hide)
+    )
+    (property "Datasheet" "" (at 151.13 80.01 0)
+      (effects (font (size 1.27 1.27)) hide)
+    )
+    (pin "1")
+    (instances
+      (project "minimouse"
+        (path "/d8fa4cba-2469-4231-847f-065b6b829f44/d17bb1c7-f68a-465e-9a17-5858ef86fc30"
+          (reference "#PWR023") (unit 1)
+        )
+      )
+    )
+  )
+  (symbol (lib_id "power:+BATT") (at 123.19 69.85 0) (unit 1)
+    (in_bom yes) (on_board yes) (dnp no) (fields_autoplaced)
+    (property "Reference" "#PWR033" (at 123.19 73.66 0)
+      (effects (font (size 1.27 1.27)) hide)
+    )
+    (property "Value" "+BATT" (at 123.19 64.77 0)
+      (effects (font (size 1.27 1.27)))
+    )
+    (property "Footprint" "" (at 123.19 69.85 0)
+      (effects (font (size 1.27 1.27)) hide)
+    )
+    (property "Datasheet" "" (at 123.19 69.85 0)
+      (effects (font (size 1.27 1.27)) hide)
+    )
+    (pin "1")
+    (instances
+      (project "minimouse"
+        (path "/d8fa4cba-2469-4231-847f-065b6b829f44/d17bb1c7-f68a-465e-9a17-5858ef86fc30"
+          (reference "#PWR033") (unit 1)
+        )
+      )
+    )
+  )
+  (symbol (lib_id "minimouse:R") (at 154.94 90.17 90) (unit 1)
+    (in_bom yes) (on_board yes) (dnp no) (fields_autoplaced)
+    (property "Reference" "R19" (at 154.94 83.82 90)
+      (effects (font (size 1.27 1.27)) hide)
+    )
+    (property "Value" "100" (at 154.94 86.36 90)
+      (effects (font (size 1.27 1.27)))
+    )
+    (property "Footprint" "Resistor_SMD:R_0603_1608Metric" (at 154.94 91.948 90)
+      (effects (font (size 1.27 1.27)) hide)
+    )
+    (property "Datasheet" "~" (at 154.94 90.17 0)
+      (effects (font (size 1.27 1.27)) hide)
+    )
+    (pin "1")
+    (pin "2")
+    (instances
+      (project "minimouse"
+        (path "/d8fa4cba-2469-4231-847f-065b6b829f44/224298a9-7d6e-4a70-a0a5-f2614895ec28"
+          (reference "R19") (unit 1)
+        )
+        (path "/d8fa4cba-2469-4231-847f-065b6b829f44/d17bb1c7-f68a-465e-9a17-5858ef86fc30"
+          (reference "R20") (unit 1)
+        )
+      )
+    )
+  )
+  (symbol (lib_id "power:GND") (at 123.19 85.09 0) (unit 1)
+    (in_bom yes) (on_board yes) (dnp no) (fields_autoplaced)
+    (property "Reference" "#PWR032" (at 123.19 91.44 0)
+      (effects (font (size 1.27 1.27)) hide)
+    )
+    (property "Value" "GND" (at 123.19 90.17 0)
+      (effects (font (size 1.27 1.27)))
+    )
+    (property "Footprint" "" (at 123.19 85.09 0)
+      (effects (font (size 1.27 1.27)) hide)
+    )
+    (property "Datasheet" "" (at 123.19 85.09 0)
+      (effects (font (size 1.27 1.27)) hide)
+    )
+    (pin "1")
+    (instances
+      (project "minimouse"
+        (path "/d8fa4cba-2469-4231-847f-065b6b829f44/d17bb1c7-f68a-465e-9a17-5858ef86fc30"
+          (reference "#PWR032") (unit 1)
+        )
+      )
+    )
+  )
+  (symbol (lib_id "power:GND") (at 130.81 97.79 0) (unit 1)
+    (in_bom yes) (on_board yes) (dnp no) (fields_autoplaced)
+    (property "Reference" "#PWR024" (at 130.81 104.14 0)
+      (effects (font (size 1.27 1.27)) hide)
+    )
+    (property "Value" "GND" (at 130.81 102.87 0)
+      (effects (font (size 1.27 1.27)))
+    )
+    (property "Footprint" "" (at 130.81 97.79 0)
+      (effects (font (size 1.27 1.27)) hide)
+    )
+    (property "Datasheet" "" (at 130.81 97.79 0)
+      (effects (font (size 1.27 1.27)) hide)
+    )
+    (pin "1")
+    (instances
+      (project "minimouse"
+        (path "/d8fa4cba-2469-4231-847f-065b6b829f44/d17bb1c7-f68a-465e-9a17-5858ef86fc30"
+          (reference "#PWR024") (unit 1)
+        )
+      )
+    )
+  )
+  (symbol (lib_id "Connector_Generic:Conn_01x04") (at 165.1 87.63 0) (unit 1)
+    (in_bom yes) (on_board yes) (dnp no) (fields_autoplaced)
+    (property "Reference" "J4" (at 167.64 87.63 0)
+      (effects (font (size 1.27 1.27)) (justify left))
+    )
+    (property "Value" "Conn_01x04" (at 167.64 90.17 0)
+      (effects (font (size 1.27 1.27)) (justify left))
+    )
+    (property "Footprint" "Connector_PinHeader_2.54mm:PinHeader_1x04_P2.54mm_Vertical" (at 165.1 87.63 0)
+      (effects (font (size 1.27 1.27)) hide)
+    )
+    (property "Datasheet" "~" (at 165.1 87.63 0)
+      (effects (font (size 1.27 1.27)) hide)
+    )
+    (pin "1")
+    (pin "4")
+    (pin "2")
+    (pin "3")
+    (instances
+      (project "minimouse"
+        (path "/d8fa4cba-2469-4231-847f-065b6b829f44/d17bb1c7-f68a-465e-9a17-5858ef86fc30"
+          (reference "J4") (unit 1)
+        )
+      )
+    )
+  )
 )

Commit message: [Debut du routage TP3]
Parts:
- removed C17: 0.1uF, Capacitor_SMD:C_0603_1608Metric, symbol minimouse:C
- renumbered R19 to R20
Connections:
- net +BATT: now also J4.2 (Pin_2); no longer J4.1 (Pin_1)
- net GND: now also J4.1 (Pin_1); no longer J4.2 (Pin_2)
Changed lines of the file:
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@@
 (kicad_sch (version 20230121) (generator eeschema)
   (paper "A4")
-  (junction (at 123.19 73.66) (diameter 0) (color 0 0 0 0)
-  )
-  (junction (at 123.19 81.28) (diameter 0) (color 0 0 0 0)
-  )
   (wire (pts (xy 123.19 81.28) (xy 123.19 85.09))
     (stroke (width 0) (type default))
@@
     (stroke (width 0) (type default))
   )
-  (wire (pts (xy 151.13 85.09) (xy 160.02 85.09))
+  (wire (pts (xy 158.75 90.17) (xy 160.02 90.17))
     (stroke (width 0) (type default))
   )
-  (wire (pts (xy 158.75 90.17) (xy 160.02 90.17))
+  (wire (pts (xy 151.13 80.01) (xy 151.13 87.63))
+    (stroke (width 0) (type default))
+  )
+  (wire (pts (xy 133.35 85.09) (xy 133.35 101.6))
     (stroke (width 0) (type default))
   )
@@
     (stroke (width 0) (type default))
   )
-  (wire (pts (xy 110.49 81.28) (xy 123.19 81.28))
+  (wire (pts (xy 151.13 87.63) (xy 160.02 87.63))
     (stroke (width 0) (type default))
   )
-  (wire (pts (xy 130.81 97.79) (xy 130.81 87.63))
-    (stroke (width 0) (type default))
-  )
-  (wire (pts (xy 151.13 80.01) (xy 151.13 85.09))
-    (stroke (width 0) (type default))
-  )
-  (wire (pts (xy 130.81 87.63) (xy 160.02 87.63))
-    (stroke (width 0) (type default))
-  )
-  (wire (pts (xy 110.49 73.66) (xy 123.19 73.66))
+  (wire (pts (xy 160.02 85.09) (xy 133.35 85.09))
     (stroke (width 0) (type default))
   )
@@
   (hierarchical_label "EXT_UART_TX" (shape output) (at 149.86 90.17 180) (fields_autoplaced)
     (effects (font (size 1.27 1.27)) (justify right))
-  )
-  (symbol (lib_id "minimouse:C") (at 110.49 77.47 0) (unit 1)
-    (in_bom yes) (on_board yes) (dnp no) (fields_autoplaced)
-    (property "Reference" "C17" (at 114.3 76.2 0)
-      (effects (font (size 1.27 1.27)) (justify left) hide)
-    )
-    (property "Value" "0.1uF" (at 114.3 78.74 0)
-      (effects (font (size 1.27 1.27)) (justify left))
-    )
-    (property "Footprint" "Capacitor_SMD:C_0603_1608Metric" (at 111.4552 81.28 0)
-      (effects (font (size 1.27 1.27)) hide)
-    )
-    (property "Datasheet" "~" (at 110.49 77.47 0)
-      (effects (font (size 1.27 1.27)) hide)
-    )
-    (pin "1")
-    (pin "2")
-    (instances
-      (project "minimouse"
-        (path "/d8fa4cba-2469-4231-847f-065b6b829f44/224298a9-7d6e-4a70-a0a5-f2614895ec28"
-          (reference "C17") (unit 1)
-        )
-        (path "/d8fa4cba-2469-4231-847f-065b6b829f44/d17bb1c7-f68a-465e-9a17-5858ef86fc30"
-          (reference "C18") (unit 1)
-        )
-      )
-    )
   )
   (symbol (lib_id "minimouse:C") (at 123.19 77.47 0) (unit 1)
@@
   (symbol (lib_id "minimouse:R") (at 154.94 90.17 90) (unit 1)
     (in_bom yes) (on_board yes) (dnp no) (fields_autoplaced)
-    (property "Reference" "R19" (at 154.94 83.82 90)
+    (property "Reference" "R20" (at 154.94 83.82 90)
       (effects (font (size 1.27 1.27)) hide)
     )
@@
     (instances
       (project "minimouse"
-        (path "/d8fa4cba-2469-4231-847f-065b6b829f44/224298a9-7d6e-4a70-a0a5-f2614895ec28"
-          (reference "R19") (unit 1)
-        )
         (path "/d8fa4cba-2469-4231-847f-065b6b829f44/d17bb1c7-f68a-465e-9a17-5858ef86fc30"
           (reference "R20") (unit 1)
@@
     )
   )
-  (symbol (lib_id "power:GND") (at 130.81 97.79 0) (unit 1)
+  (symbol (lib_id "power:GND") (at 133.35 101.6 0) (unit 1)
     (in_bom yes) (on_board yes) (dnp no) (fields_autoplaced)
-    (property "Reference" "#PWR024" (at 130.81 104.14 0)
+    (property "Reference" "#PWR024" (at 133.35 107.95 0)
       (effects (font (size 1.27 1.27)) hide)
     )
-    (property "Value" "GND" (at 130.81 102.87 0)
+    (property "Value" "GND" (at 133.35 106.68 0)
       (effects (font (size 1.27 1.27)))
     )
-    (property "Footprint" "" (at 130.81 97.79 0)
+    (property "Footprint" "" (at 133.35 101.6 0)
       (effects (font (size 1.27 1.27)) hide)
     )
-    (property "Datasheet" "" (at 130.81 97.79 0)
+    (property "Datasheet" "" (at 133.35 101.6 0)
       (effects (font (size 1.27 1.27)) hide)
     )
