File: mm_motor.kicad_sch (KiCad schematic)
At the start: 1 part, among them M1 N20_encoder

Commit message: fin tp2
Parts:
- added C15: 2.2uF, Capacitor_SMD:C_0603_1608Metric, symbol minimouse:C
- added C17: 0.1uF, Capacitor_SMD:C_0603_1608Metric, symbol minimouse:C
- added J2: Conn_01x06, Connector_PinHeader_2.54mm:PinHeader_1x06_P2.54mm_Vertical, symbol Connector_Generic:Conn_01x06
- added R19 (x2): 100, Resistor_SMD:R_0603_1608Metric, symbol minimouse:R
Connections:
- net C1: now also R19.1
- net C2: now also R19.1
- net MA: now also J2.1 (Pin_1)
- net MB: now also J2.6 (Pin_6)
- new net: J2.3 (Pin_3), R19.2
- new net: J2.4 (Pin_4), R19.2
- new net +BATT: C15.1, C17.1, J2.5 (Pin_5)
- new net GND: C15.2, C17.2, J2.2 (Pin_2)

Commit message: [Debut du routage TP3]
Parts:
- removed C17: 0.1uF, Capacitor_SMD:C_0603_1608Metric, symbol minimouse:C
- renumbered R19 to R21, R19 to R23
Changed lines of the file:
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@@
   (junction (at 102.87 96.52) (diameter 0) (color 0 0 0 0)
   )
-  (junction (at 102.87 106.68) (diameter 0) (color 0 0 0 0)
-  )
-  (junction (at 102.87 99.06) (diameter 0) (color 0 0 0 0)
-  )
   (wire (pts (xy 133.35 91.44) (xy 143.51 91.44))
     (stroke (width 0) (type default))
@@
     (stroke (width 0) (type default))
   )
+  (wire (pts (xy 109.22 115.57) (xy 109.22 88.9))
+    (stroke (width 0) (type default))
+  )
   (wire (pts (xy 143.51 96.52) (xy 102.87 96.52))
     (stroke (width 0) (type default))
   )
+  (wire (pts (xy 109.22 88.9) (xy 143.51 88.9))
+    (stroke (width 0) (type default))
+  )
   (wire (pts (xy 102.87 96.52) (xy 102.87 99.06))
     (stroke (width 0) (type default))
   )
-  (wire (pts (xy 91.44 99.06) (xy 102.87 99.06))
-    (stroke (width 0) (type default))
-  )
   (wire (pts (xy 133.35 93.98) (xy 143.51 93.98))
     (stroke (width 0) (type default))
@@
     (stroke (width 0) (type default))
   )
-  (wire (pts (xy 91.44 106.68) (xy 102.87 106.68))
-    (stroke (width 0) (type default))
-  )
   (wire (pts (xy 102.87 96.52) (xy 102.87 77.47))
-    (stroke (width 0) (type default))
-  )
-  (wire (pts (xy 107.95 88.9) (xy 143.51 88.9))
     (stroke (width 0) (type default))
   )
@@
   (symbol (lib_id "minimouse:R") (at 129.54 91.44 90) (unit 1)
     (in_bom yes) (on_board yes) (dnp no) (fields_autoplaced)
-    (property "Reference" "R19" (at 129.54 85.09 90)
+    (property "Reference" "R21" (at 129.54 85.09 90)
       (effects (font (size 1.27 1.27)) hide)
     )
@@
     (instances
       (project "minimouse"
-        (path "/d8fa4cba-2469-4231-847f-065b6b829f44/224298a9-7d6e-4a70-a0a5-f2614895ec28"
-          (reference "R19") (unit 1)
-        )
         (path "/d8fa4cba-2469-4231-847f-065b6b829f44/7f113667-692a-4f4d-b16f-621d32f3f136"
           (reference "R21") (unit 1)
@@
   (symbol (lib_id "minimouse:R") (at 129.54 93.98 90) (unit 1)
     (in_bom yes) (on_board yes) (dnp no) (fields_autoplaced)
-    (property "Reference" "R19" (at 129.54 87.63 90)
+    (property "Reference" "R23" (at 129.54 87.63 90)
       (effects (font (size 1.27 1.27)) hide)
     )
@@
     (instances
       (project "minimouse"
-        (path "/d8fa4cba-2469-4231-847f-065b6b829f44/224298a9-7d6e-4a70-a0a5-f2614895ec28"
-          (reference "R19") (unit 1)
-        )
         (path "/d8fa4cba-2469-4231-847f-065b6b829f44/7f113667-692a-4f4d-b16f-621d32f3f136"
           (reference "R23") (unit 1)
@@
     )
   )
-  (symbol (lib_id "power:GND") (at 107.95 88.9 0) (unit 1)
-    (in_bom yes) (on_board yes) (dnp no) (fields_autoplaced)
-    (property "Reference" "#PWR019" (at 107.95 95.25 0)
-      (effects (font (size 1.27 1.27)) hide)
-    )
-    (property "Value" "GND" (at 107.95 93.98 0)
-      (effects (font (size 1.27 1.27)))
-    )
-    (property "Footprint" "" (at 107.95 88.9 0)
-      (effects (font (size 1.27 1.27)) hide)
-    )
-    (property "Datasheet" "" (at 107.95 88.9 0)
+  (symbol (lib_id "power:GND") (at 109.22 115.57 0) (unit 1)
+    (in_bom yes) (on_board yes) (dnp no) (fields_autoplaced)
+    (property "Reference" "#PWR019" (at 109.22 121.92 0)
+      (effects (font (size 1.27 1.27)) hide)
+    )
+    (property "Value" "GND" (at 109.22 120.65 0)
+      (effects (font (size 1.27 1.27)))
+    )
+    (property "Footprint" "" (at 109.22 115.57 0)
+      (effects (font (size 1.27 1.27)) hide)
+    )
+    (property "Datasheet" "" (at 109.22 115.57 0)
       (effects (font (size 1.27 1.27)) hide)
     )
@@
         )
       )
-    )
-  )
-  (symbol (lib_id "minimouse:C") (at 91.44 102.87 0) (unit 1)
-    (in_bom yes) (on_board yes) (dnp no) (fields_autoplaced)
-    (property "Reference" "C17" (at 95.25 101.6 0)
-      (effects (font (size 1.27 1.27)) (justify left) hide)
-    )
-    (property "Value" "0.1uF" (at 95.25 104.14 0)
-      (effects (font (size 1.27 1.27)) (justify left))
-    )
-    (property "Footprint" "Capacitor_SMD:C_0603_1608Metric" (at 92.4052 106.68 0)
-      (effects (font (size 1.27 1.27)) hide)
-    )
-    (property "Datasheet" "~" (at 91.44 102.87 0)
-      (effects (font (size 1.27 1.27)) hide)
-    )
-    (pin "1")
-    (pin "2")
-    (instances
-      (project "minimouse"
-        (path "/d8fa4cba-2469-4231-847f-065b6b829f44/224298a9-7d6e-4a70-a0a5-f2614895ec28"
-          (reference "C17") (unit 1)
-        )
-        (path "/d8fa4cba-2469-4231-847f-065b6b829f44/7f113667-692a-4f4d-b16f-621d32f3f136"
-          (reference "C19") (unit 1)
-        )
-        (path "/d8fa4cba-2469-4231-847f-065b6b829f44/3975acd0-18ad-47bc-9ce1-d8c4d864aafe"
-          (reference "C20") (unit 1)
-        )
-      )
