File: mm_ultrasonic_sensor.kicad_sch (KiCad schematic)
At the start: 0 parts

Commit message: fin tp2
Parts:
- added C13: 2.2uF, Capacitor_SMD:C_0603_1608Metric, symbol minimouse:C
- added C17: 0.1uF, Capacitor_SMD:C_0603_1608Metric, symbol minimouse:C
- added R19: 100, Resistor_SMD:R_0603_1608Metric, symbol minimouse:R
- added U4: HC-SR04, minimouse:HC-SR04, symbol minimouse:HC-SR04
Connections:
- net SONAR_ECHO: now also R19.1
- net SONAR_TRIGGER: now also U4.2 (TRIG)
- new net: R19.2, U4.3 (ECHO)
- new net +BATT: C13.1, C17.1, U4.4 (VCC)
- new net GND: C13.2, C17.2, U4.1 (GND)
Changed lines of the file:
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@@
 (kicad_sch (version 20230121) (generator eeschema)
   (paper "A4")
-  (hierarchical_label "SONAR_TRIGGER" (shape input) (at 109.22 88.9 180) (fields_autoplaced)
+  (junction (at 110.49 63.5) (diameter 0) (color 0 0 0 0)
+  )
+  (junction (at 110.49 71.12) (diameter 0) (color 0 0 0 0)
+  )
+  (wire (pts (xy 148.59 73.66) (xy 148.59 78.74))
+    (stroke (width 0) (type default))
+  )
+  (wire (pts (xy 110.49 59.69) (xy 110.49 63.5))
+    (stroke (width 0) (type default))
+  )
+  (wire (pts (xy 97.79 71.12) (xy 110.49 71.12))
+    (stroke (width 0) (type default))
+  )
+  (wire (pts (xy 109.22 90.17) (xy 119.38 90.17))
+    (stroke (width 0) (type default))
+  )
+  (wire (pts (xy 127 90.17) (xy 138.43 90.17))
+    (stroke (width 0) (type default))
+  )
+  (wire (pts (xy 110.49 71.12) (xy 110.49 74.93))
+    (stroke (width 0) (type default))
+  )
+  (wire (pts (xy 148.59 99.06) (xy 148.59 105.41))
+    (stroke (width 0) (type default))
+  )
+  (wire (pts (xy 97.79 63.5) (xy 110.49 63.5))
+    (stroke (width 0) (type default))
+  )
+  (wire (pts (xy 109.22 87.63) (xy 138.43 87.63))
+    (stroke (width 0) (type default))
+  )
+  (hierarchical_label "SONAR_TRIGGER" (shape input) (at 109.22 87.63 180) (fields_autoplaced)
     (effects (font (size 1.27 1.27)) (justify right))
   )
-  (hierarchical_label "SONAR_ECHO" (shape output) (at 109.22 91.44 180) (fields_autoplaced)
+  (hierarchical_label "SONAR_ECHO" (shape output) (at 109.22 90.17 180) (fields_autoplaced)
     (effects (font (size 1.27 1.27)) (justify right))
   )
+  (symbol (lib_id "power:+BATT") (at 148.59 73.66 0) (unit 1)
+    (in_bom yes) (on_board yes) (dnp no) (fields_autoplaced)
+    (property "Reference" "#PWR034" (at 148.59 77.47 0)
+      (effects (font (size 1.27 1.27)) hide)
+    )
+    (property "Value" "+BATT" (at 148.59 68.58 0)
+      (effects (font (size 1.27 1.27)))
+    )
+    (property "Footprint" "" (at 148.59 73.66 0)
+      (effects (font (size 1.27 1.27)) hide)
+    )
+    (property "Datasheet" "" (at 148.59 73.66 0)
+      (effects (font (size 1.27 1.27)) hide)
+    )
+    (pin "1")
+    (instances
+      (project "minimouse"
+        (path "/d8fa4cba-2469-4231-847f-065b6b829f44/224298a9-7d6e-4a70-a0a5-f2614895ec28"
+          (reference "#PWR034") (unit 1)
+        )
+      )
+    )
+  )
+  (symbol (lib_id "minimouse:C") (at 110.49 67.31 0) (unit 1)
+    (in_bom yes) (on_board yes) (dnp no) (fields_autoplaced)
+    (property "Reference" "C13" (at 114.3 66.04 0)
+      (effects (font (size 1.27 1.27)) (justify left) hide)
+    )
+    (property "Value" "2.2uF" (at 114.3 68.58 0)
+      (effects (font (size 1.27 1.27)) (justify left))
+    )
+    (property "Footprint" "Capacitor_SMD:C_0603_1608Metric" (at 111.4552 71.12 0)
+      (effects (font (size 1.27 1.27)) hide)
+    )
+    (property "Datasheet" "~" (at 110.49 67.31 0)
+      (effects (font (size 1.27 1.27)) hide)
+    )
+    (pin "1")
+    (pin "2")
+    (instances
+      (project "minimouse"
+        (path "/d8fa4cba-2469-4231-847f-065b6b829f44/d17bb1c7-f68a-465e-9a17-5858ef86fc30"
+          (reference "C13") (unit 1)
+        )
+        (path "/d8fa4cba-2469-4231-847f-065b6b829f44/224298a9-7d6e-4a70-a0a5-f2614895ec28"
+          (reference "C16") (unit 1)
+        )
+      )
+    )
+  )
+  (symbol (lib_id "power:+BATT") (at 110.49 59.69 0) (unit 1)
+    (in_bom yes) (on_board yes) (dnp no) (fields_autoplaced)
+    (property "Reference" "#PWR033" (at 110.49 63.5 0)
+      (effects (font (size 1.27 1.27)) hide)
+    )
+    (property "Value" "+BATT" (at 110.49 54.61 0)
+      (effects (font (size 1.27 1.27)))
+    )
+    (property "Footprint" "" (at 110.49 59.69 0)
+      (effects (font (size 1.27 1.27)) hide)
+    )
+    (property "Datasheet" "" (at 110.49 59.69 0)
+      (effects (font (size 1.27 1.27)) hide)
+    )
+    (pin "1")
+    (instances
+      (project "minimouse"
+        (path "/d8fa4cba-2469-4231-847f-065b6b829f44/d17bb1c7-f68a-465e-9a17-5858ef86fc30"
+          (reference "#PWR033") (unit 1)
+        )
+        (path "/d8fa4cba-2469-4231-847f-065b6b829f44/224298a9-7d6e-4a70-a0a5-f2614895ec28"
+          (reference "#PWR035") (unit 1)
+        )
+      )
+    )
+  )
+  (symbol (lib_id "power:GND") (at 110.49 74.93 0) (unit 1)
+    (in_bom yes) (on_board yes) (dnp no) (fields_autoplaced)
+    (property "Reference" "#PWR032" (at 110.49 81.28 0)
+      (effects (font (size 1.27 1.27)) hide)
+    )
+    (property "Value" "GND" (at 110.49 80.01 0)
+      (effects (font (size 1.27 1.27)))
+    )
+    (property "Footprint" "" (at 110.49 74.93 0)
+      (effects (font (size 1.27 1.27)) hide)
+    )
+    (property "Datasheet" "" (at 110.49 74.93 0)
+      (effects (font (size 1.27 1.27)) hide)
+    )
+    (pin "1")
+    (instances
+      (project "minimouse"
+        (path "/d8fa4cba-2469-4231-847f-065b6b829f44/d17bb1c7-f68a-465e-9a17-5858ef86fc30"
+          (reference "#PWR032") (unit 1)
+        )
+        (path "/d8fa4cba-2469-4231-847f-065b6b829f44/224298a9-7d6e-4a70-a0a5-f2614895ec28"
+          (reference "#PWR040") (unit 1)
+        )
+      )
+    )
+  )
+  (symbol (lib_id "minimouse:R") (at 123.19 90.17 90) (unit 1)
+    (in_bom yes) (on_board yes) (dnp no) (fields_autoplaced)
+    (property "Reference" "R19" (at 123.19 83.82 90)
+      (effects (font (size 1.27 1.27)) hide)
+    )
+    (property "Value" "100" (at 123.19 86.36 90)
+      (effects (font (size 1.27 1.27)))
+    )
+    (property "Footprint" "Resistor_SMD:R_0603_1608Metric" (at 123.19 91.948 90)
+      (effects (font (size 1.27 1.27)) hide)
+    )
+    (property "Datasheet" "~" (at 123.19 90.17 0)
+      (effects (font (size 1.27 1.27)) hide)
+    )
+    (pin "1")
+    (pin "2")
+    (instances
+      (project "minimouse"
+        (path "/d8fa4cba-2469-4231-847f-065b6b829f44/224298a9-7d6e-4a70-a0a5-f2614895ec28"
+          (reference "R19") (unit 1)
+        )
+      )
+    )
+  )
+  (symbol (lib_id "minimouse:C") (at 97.79 67.31 0) (unit 1)
+    (in_bom yes) (on_board yes) (dnp no) (fields_autoplaced)
+    (property "Reference" "C17" (at 101.6 66.04 0)
+      (effects (font (size 1.27 1.27)) (justify left) hide)
+    )
+    (property "Value" "0.1uF" (at 101.6 68.58 0)
+      (effects (font (size 1.27 1.27)) (justify left))
+    )
+    (property "Footprint" "Capacitor_SMD:C_0603_1608Metric" (at 98.7552 71.12 0)
+      (effects (font (size 1.27 1.27)) hide)
+    )
+    (property "Datasheet" "~" (at 97.79 67.31 0)
+      (effects (font (size 1.27 1.27)) hide)
+    )
+    (pin "1")
+    (pin "2")
+    (instances
+      (project "minimouse"
+        (path "/d8fa4cba-2469-4231-847f-065b6b829f44/224298a9-7d6e-4a70-a0a5-f2614895ec28"
+          (reference "C17") (unit 1)
+        )
+      )
+    )
+  )
+  (symbol (lib_id "power:GND") (at 148.59 105.41 0) (unit 1)
+    (in_bom yes) (on_board yes) (dnp no) (fields_autoplaced)
+    (property "Reference" "#PWR041" (at 148.59 111.76 0)
+      (effects (font (size 1.27 1.27)) hide)
+    )
+    (property "Value" "GND" (at 148.59 110.49 0)
+      (effects (font (size 1.27 1.27)))
+    )
+    (property "Footprint" "" (at 148.59 105.41 0)
+      (effects (font (size 1.27 1.27)) hide)
+    )
+    (property "Datasheet" "" (at 148.59 105.41 0)
+      (effects (font (size 1.27 1.27)) hide)
+    )
+    (pin "1")
+    (instances
+      (project "minimouse"
+        (path "/d8fa4cba-2469-4231-847f-065b6b829f44/224298a9-7d6e-4a70-a0a5-f2614895ec28"
+          (reference "#PWR041") (unit 1)
+        )
+      )
+    )
+  )
+  (symbol (lib_id "minimouse:HC-SR04") (at 148.59 88.9 0) (unit 1)
+    (in_bom yes) (on_board yes) (dnp no) (fields_autoplaced)
+    (property "Reference" "U4" (at 161.29 87.63 0)
+      (effects (font (size 1.27 1.27)) (justify left))
+    )
+    (property "Value" "HC-SR04" (at 161.29 90.17 0)
+      (effects (font (size 1.27 1.27)) (justify left))
+    )
+    (property "Footprint" "minimouse:HC-SR04" (at 148.59 88.9 0)
+      (effects (font (size 1.27 1.27)) hide)
+    )
+    (property "Datasheet" "" (at 148.59 88.9 0)
+      (effects (font (size 1.27 1.27)) hide)
+    )
+    (pin "3")
+    (pin "2")
+    (pin "4")
+    (pin "1")
+    (instances
+      (project "minimouse"
+        (path "/d8fa4cba-2469-4231-847f-065b6b829f44/224298a9-7d6e-4a70-a0a5-f2614895ec28"
+          (reference "U4") (unit 1)
+        )
+      )
+    )
+  )
 )

Commit message: [Debut du routage TP3]
Parts:
- removed C17: 0.1uF, Capacitor_SMD:C_0603_1608Metric, symbol minimouse:C
- renumbered C13 to C16
Changed lines of the file:
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@@
 (kicad_sch (version 20230121) (generator eeschema)
   (paper "A4")
-  (junction (at 110.49 63.5) (diameter 0) (color 0 0 0 0)
-  )
-  (junction (at 110.49 71.12) (diameter 0) (color 0 0 0 0)
-  )
   (wire (pts (xy 148.59 73.66) (xy 148.59 78.74))
     (stroke (width 0) (type default))
   )
   (wire (pts (xy 110.49 59.69) (xy 110.49 63.5))
-    (stroke (width 0) (type default))
-  )
-  (wire (pts (xy 97.79 71.12) (xy 110.49 71.12))
     (stroke (width 0) (type default))
   )
@@
   )
   (wire (pts (xy 148.59 99.06) (xy 148.59 105.41))
-    (stroke (width 0) (type default))
-  )
-  (wire (pts (xy 97.79 63.5) (xy 110.49 63.5))
     (stroke (width 0) (type default))
   )
@@
   (symbol (lib_id "minimouse:C") (at 110.49 67.31 0) (unit 1)
     (in_bom yes) (on_board yes) (dnp no) (fields_autoplaced)
-    (property "Reference" "C13" (at 114.3 66.04 0)
+    (property "Reference" "C16" (at 114.3 66.04 0)
       (effects (font (size 1.27 1.27)) (justify left) hide)
     )
@@
     (instances
       (project "minimouse"
-        (path "/d8fa4cba-2469-4231-847f-065b6b829f44/d17bb1c7-f68a-465e-9a17-5858ef86fc30"
-          (reference "C13") (unit 1)
-        )
         (path "/d8fa4cba-2469-4231-847f-065b6b829f44/224298a9-7d6e-4a70-a0a5-f2614895ec28"
           (reference "C16") (unit 1)
@@
   (symbol (lib_id "power:+BATT") (at 110.49 59.69 0) (unit 1)
     (in_bom yes) (on_board yes) (dnp no) (fields_autoplaced)
-    (property "Reference" "#PWR033" (at 110.49 63.5 0)
+    (property "Reference" "#PWR035" (at 110.49 63.5 0)
       (effects (font (size 1.27 1.27)) hide)
     )
@@
     (instances
       (project "minimouse"
-        (path "/d8fa4cba-2469-4231-847f-065b6b829f44/d17bb1c7-f68a-465e-9a17-5858ef86fc30"
-          (reference "#PWR033") (unit 1)
-        )
         (path "/d8fa4cba-2469-4231-847f-065b6b829f44/224298a9-7d6e-4a70-a0a5-f2614895ec28"
           (reference "#PWR035") (unit 1)
@@
   (symbol (lib_id "power:GND") (at 110.49 74.93 0) (unit 1)
     (in_bom yes) (on_board yes) (dnp no) (fields_autoplaced)
-    (property "Reference" "#PWR032" (at 110.49 81.28 0)
+    (property "Reference" "#PWR040" (at 110.49 81.28 0)
       (effects (font (size 1.27 1.27)) hide)
     )
@@
     (instances
       (project "minimouse"
-        (path "/d8fa4cba-2469-4231-847f-065b6b829f44/d17bb1c7-f68a-465e-9a17-5858ef86fc30"
-          (reference "#PWR032") (unit 1)
-        )
         (path "/d8fa4cba-2469-4231-847f-065b6b829f44/224298a9-7d6e-4a70-a0a5-f2614895ec28"
           (reference "#PWR040") (unit 1)
@@
         )
       )
-    )
-  )
-  (symbol (lib_id "minimouse:C") (at 97.79 67.31 0) (unit 1)
-    (in_bom yes) (on_board yes) (dnp no) (fields_autoplaced)
-    (property "Reference" "C17" (at 101.6 66.04 0)
-      (effects (font (size 1.27 1.27)) (justify left) hide)
-    )
-    (property "Value" "0.1uF" (at 101.6 68.58 0)
-      (effects (font (size 1.27 1.27)) (justify left))
-    )
-    (property "Footprint" "Capacitor_SMD:C_0603_1608Metric" (at 98.7552 71.12 0)
-      (effects (font (size 1.27 1.27)) hide)
-    )
-    (property "Datasheet" "~" (at 97.79 67.31 0)
-      (effects (font (size 1.27 1.27)) hide)
-    )
-    (pin "1")
-    (pin "2")
-    (instances
-      (project "minimouse"
-        (path "/d8fa4cba-2469-4231-847f-065b6b829f44/224298a9-7d6e-4a70-a0a5-f2614895ec28"
-          (reference "C17") (unit 1)
-        )
-      )
