File: mm_motor_control.kicad_sch (KiCad schematic)
At the start: 0 parts

Commit message: fin tp2
Parts:
- added C10: 10n, Capacitor_SMD:C_0603_1608Metric, symbol minimouse:C
- added C7: 2.2uF, Capacitor_SMD:C_0603_1608Metric, symbol minimouse:C
- added C8: 22n, Capacitor_SMD:C_0603_1608Metric, symbol minimouse:C
- added C9: 1n, Capacitor_SMD:C_0603_1608Metric, symbol minimouse:C
- added R10: 1k, Resistor_SMD:R_0603_1608Metric, symbol minimouse:R
- added R11: 47k, Resistor_SMD:R_0603_1608Metric, symbol minimouse:R
- added R12, R13: 18k, Resistor_SMD:R_0603_1608Metric, symbol minimouse:R
- added R14, R15: 10k, Resistor_SMD:R_0603_1608Metric, symbol minimouse:R
- added R16, R17: 330m, Resistor_SMD:R_2512_6332Metric, symbol minimouse:R
- added R19: 100, Resistor_SMD:R_0603_1608Metric, symbol minimouse:R
- added U2: STSPIN240, Package_DFN_QFN:VQFN-16-1EP_3x3mm_P0.5mm_EP1.8x1.8mm, symbol Driver_Motor:STSPIN240
Connections:
- net EN: now also R12.1
- net FAULT: now also R19.1
- net OUT_A1: now also U2.3 (OUTA1)
- net OUT_A2: now also U2.5 (OUTA2)
- net OUT_B1: now also U2.10 (OUTB1)
- net OUT_B2: now also U2.8 (OUTB2)
- net PHASE_A: now also U2.1 (PHA)
- net PHASE_B: now also U2.15 (PHB)
- net PWM_A: now also U2.2 (PWMA)
- net PWM_B: now also U2.16 (PWMB)
- net STBY/RESET: now also C9.1, R13.1, U2.14 (STBY/RESET)
- new net: C10.1, R12.2, R19.2, U2.13 (EN/FLT)
- new net: R17.1, U2.4 (SENSEA)
- new net: R16.1, U2.9 (SENSEB)
- new net: C8.1, R10.2
- new net +3.3V: R13.2
- new net +BATT: C7.1, R14.1, U2.6 (VS)
- new net GND: C10.2, C7.2, C8.2, C9.2, R11.2, R15.2, R16.2, R17.2, U2.17 (EPAD), U2.7 (GND)
- new net REF: R14.2, R15.1, U2.11 (REF)
- new net TOFF: R10.1, R11.1, U2.12 (TOFF)

Commit message: [Debut du routage TP3]
Parts:
- removed C9: 1n, Capacitor_SMD:C_0603_1608Metric, symbol minimouse:C
- removed R13: 18k, Resistor_SMD:R_0603_1608Metric, symbol minimouse:R
- renumbered R19 to R25
Changed lines of the file:
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@@
 (kicad_sch (version 20230121) (generator eeschema)
   (paper "A4")
-  (junction (at 82.55 115.57) (diameter 0) (color 0 0 0 0)
-  )
   (junction (at 118.11 124.46) (diameter 0) (color 0 0 0 0)
   )
@@
     (stroke (width 0) (type default))
   )
-  (wire (pts (xy 82.55 113.03) (xy 82.55 115.57))
-    (stroke (width 0) (type default))
-  )
   (wire (pts (xy 153.67 107.95) (xy 153.67 110.49))
     (stroke (width 0) (type default))
@@
     (stroke (width 0) (type default))
   )
-  (wire (pts (xy 82.55 125.73) (xy 82.55 134.62))
-    (stroke (width 0) (type default))
-  )
   (wire (pts (xy 118.11 87.63) (xy 118.11 88.9))
     (stroke (width 0) (type default))
@@
     (stroke (width 0) (type default))
   )
-  (wire (pts (xy 60.96 115.57) (xy 82.55 115.57))
-    (stroke (width 0) (type default))
-  )
   (wire (pts (xy 168.91 90.17) (xy 198.12 90.17))
     (stroke (width 0) (type default))
@@
     (stroke (width 0) (type default))
   )
-  (wire (pts (xy 82.55 115.57) (xy 82.55 118.11))
-    (stroke (width 0) (type default))
-  )
   (wire (pts (xy 168.91 95.25) (xy 175.26 95.25))
     (stroke (width 0) (type default))
@@
     (stroke (width 0) (type default))
   )
-  (wire (pts (xy 82.55 115.57) (xy 87.63 115.57))
-    (stroke (width 0) (type default))
-  )
   (wire (pts (xy 114.3 83.82) (xy 140.97 83.82))
     (stroke (width 0) (type default))
@@
     (stroke (width 0) (type default))
   )
-  (wire (pts (xy 128.27 95.25) (xy 140.97 95.25))
+  (wire (pts (xy 127 95.25) (xy 140.97 95.25))
     (stroke (width 0) (type default))
   )
@@
   (wire (pts (xy 87.63 87.63) (xy 93.98 87.63))
     (stroke (width 0) (type default))
-  )
-  (label "STBY{slash}RESET" (at 128.27 95.25 0) (fields_autoplaced)
-    (effects (font (size 1.27 1.27)) (justify left bottom))
-  )
-  (label "STBY{slash}RESET" (at 87.63 115.57 0) (fields_autoplaced)
-    (effects (font (size 1.27 1.27)) (justify left bottom))
   )
   (label "TOFF" (at 118.11 120.65 0) (fields_autoplaced)
@@
     (effects (font (size 1.27 1.27)) (justify left))
   )
-  (hierarchical_label "STBY{slash}RESET" (shape input) (at 60.96 115.57 180) (fields_autoplaced)
+  (hierarchical_label "STBY{slash}RESET" (shape input) (at 127 95.25 180) (fields_autoplaced)
     (effects (font (size 1.27 1.27)) (justify right))
   )
@@
     )
   )
-  (symbol (lib_id "minimouse:C") (at 82.55 121.92 0) (unit 1)
-    (in_bom yes) (on_board yes) (dnp no) (fields_autoplaced)
-    (property "Reference" "C9" (at 86.36 120.65 0)
-      (effects (font (size 1.27 1.27)) (justify left) hide)
-    )
-    (property "Value" "1n" (at 86.36 123.19 0)
-      (effects (font (size 1.27 1.27)) (justify left))
-    )
-    (property "Footprint" "Capacitor_SMD:C_0603_1608Metric" (at 83.5152 125.73 0)
-      (effects (font (size 1.27 1.27)) hide)
-    )
-    (property "Datasheet" "~" (at 82.55 121.92 0)
-      (effects (font (size 1.27 1.27)) hide)
-    )
-    (pin "1")
-    (pin "2")
-    (instances
-      (project "minimouse"
-        (path "/d8fa4cba-2469-4231-847f-065b6b829f44/0999fad3-9a14-4ede-b729-a71c3dbbdf8e"
-          (reference "C9") (unit 1)
-        )
-      )
-    )
-  )
-  (symbol (lib_id "power:GND") (at 82.55 134.62 0) (unit 1)
-    (in_bom yes) (on_board yes) (dnp no) (fields_autoplaced)
-    (property "Reference" "#PWR013" (at 82.55 140.97 0)
-      (effects (font (size 1.27 1.27)) hide)
-    )
-    (property "Value" "GND" (at 82.55 139.7 0)
-      (effects (font (size 1.27 1.27)))
-    )
-    (property "Footprint" "" (at 82.55 134.62 0)
-      (effects (font (size 1.27 1.27)) hide)
-    )
-    (property "Datasheet" "" (at 82.55 134.62 0)
-      (effects (font (size 1.27 1.27)) hide)
-    )
-    (pin "1")
-    (instances
-      (project "minimouse"
-        (path "/d8fa4cba-2469-4231-847f-065b6b829f44/0999fad3-9a14-4ede-b729-a71c3dbbdf8e"
-          (reference "#PWR013") (unit 1)
-        )
-      )
-    )
-  )
   (symbol (lib_id "power:GND") (at 189.23 104.14 0) (unit 1)
     (in_bom yes) (on_board yes) (dnp no) (fields_autoplaced)
@@
     )
   )
-  (symbol (lib_id "minimouse:R") (at 82.55 109.22 180) (unit 1)
-    (in_bom yes) (on_board yes) (dnp no) (fields_autoplaced)
-    (property "Reference" "R13" (at 85.09 107.95 0)
-      (effects (font (size 1.27 1.27)) (justify right) hide)
-    )
-    (property "Value" "18k" (at 85.09 110.49 0)
-      (effects (font (size 1.27 1.27)) (justify right))
-    )
-    (property "Footprint" "Resistor_SMD:R_0603_1608Metric" (at 84.328 109.22 90)
-      (effects (font (size 1.27 1.27)) hide)
-    )
-    (property "Datasheet" "~" (at 82.55 109.22 0)
-      (effects (font (size 1.27 1.27)) hide)
-    )
-    (pin "2")
-    (pin "1")
-    (instances
-      (project "minimouse"
-        (path "/d8fa4cba-2469-4231-847f-065b6b829f44/0999fad3-9a14-4ede-b729-a71c3dbbdf8e"
-          (reference "R13") (unit 1)
-        )
-      )
-    )
-  )
   (symbol (lib_id "power:+BATT") (at 57.15 123.19 0) (unit 1)
     (in_bom yes) (on_board yes) (dnp no) (fields_autoplaced)
@@
   (symbol (lib_id "minimouse:R") (at 83.82 87.63 90) (unit 1)
     (in_bom yes) (on_board yes) (dnp no) (fields_autoplaced)
-    (property "Reference" "R19" (at 83.82 81.28 90)
+    (property "Reference" "R25" (at 83.82 81.28 90)
       (effects (font (size 1.27 1.27)) hide)
     )
@@
     (instances
       (project "minimouse"
-        (path "/d8fa4cba-2469-4231-847f-065b6b829f44/224298a9-7d6e-4a70-a0a5-f2614895ec28"
-          (reference "R19") (unit 1)
-        )
         (path "/d8fa4cba-2469-4231-847f-065b6b829f44/0999fad3-9a14-4ede-b729-a71c3dbbdf8e"
           (reference "R25") (unit 1)

Commit message: [Routage PCB]
Parts:
- removed C7: 2.2uF, Capacitor_SMD:C_0603_1608Metric, symbol minimouse:C
- added C9: 2.2uF, Capacitor_SMD:C_0603_1608Metric, symbol minimouse:C
Connections:
- net +BATT: now also C9.1
- net GND: now also C9.2
