File: minimouse.kicad_pcb (KiCad board)
At the start: 2 copper layers, 90 x 85 mm, 22 parts, among them J1 Conn_ARM_JTAG_SWD_10, J5 Conn_01x02, M1 N20_encoder, M2 N20_encoder, U1 STM32F030C8Tx, U4 HC-SR04

Commit message: [Debut du routage TP3]
Parts:
- added C10: 10n, Capacitor_SMD:C_0603_1608Metric, F.Cu at (149.9, 101.9)
- added C11: 2.2uF, Capacitor_SMD:C_0603_1608Metric, F.Cu at (177.8, 89.2)
- added C12: 2.2uF, Capacitor_SMD:C_0603_1608Metric, F.Cu at (185.8, 89.2)
- added C13: 2.2uF, Capacitor_SMD:C_0603_1608Metric, F.Cu at (123.4, 79.6)
- added C14: 2.2uF, Capacitor_SMD:C_0603_1608Metric, F.Cu at (175.3, 100.1)
- added C15: 2.2uF, Capacitor_SMD:C_0603_1608Metric, F.Cu at (129.9, 100.4)
- added C16: 2.2uF, Capacitor_SMD:C_0603_1608Metric, F.Cu at (153.8, 72.3)
- added C8: 22n, Capacitor_SMD:C_0603_1608Metric, F.Cu at (161.8, 101.2)
- added C9: 2.2uF, Capacitor_SMD:C_0603_1608Metric, F.Cu at (149.0, 110.4)
- added D1: LED, LED_SMD:LED_0603_1608Metric, F.Cu at (186.5, 91.7)
- added J2: Conn_01x06, Connector_PinHeader_2.54mm:PinHeader_1x06_P2.54mm_Vertical, F.Cu at (165.2, 104.5)
- added J3: Conn_01x06, Connector_PinHeader_2.54mm:PinHeader_1x06_P2.54mm_Vertical, F.Cu at (123.6, 104.8)
- added J4: Conn_01x04, Connector_PinHeader_2.54mm:PinHeader_1x04_P2.54mm_Vertical, F.Cu at (119.5, 77.2)
- added R10: 1k, Resistor_SMD:R_0603_1608Metric, F.Cu at (158.6, 101.2)
- added R11: 47k, Resistor_SMD:R_0603_1608Metric, F.Cu at (160.3, 99.4)
- added R12: 18k, Resistor_SMD:R_0603_1608Metric, F.Cu at (153.0, 102.7)
- added R14: 10k, Resistor_SMD:R_0603_1608Metric, F.Cu at (154.9, 109.2)
- added R15: 10k, Resistor_SMD:R_0603_1608Metric, F.Cu at (155.0, 110.8)
- added R16: 330m, Resistor_SMD:R_2512_6332Metric, F.Cu at (157.0, 115.0)
- added R17: 330m, Resistor_SMD:R_2512_6332Metric, F.Cu at (142.2, 114.9)
- added R18: 330, Resistor_SMD:R_0603_1608Metric, F.Cu at (186.5, 94.9)
- added R19: 100, Resistor_SMD:R_0603_1608Metric, F.Cu at (151.3, 72.3)
- added R20: 100, Resistor_SMD:R_0603_1608Metric, F.Cu at (123.5, 82.2)
- added R21: 100, Resistor_SMD:R_0603_1608Metric, F.Cu at (170.4, 100.0)
- added R22: 100, Resistor_SMD:R_0603_1608Metric, F.Cu at (132.8, 100.3)
- added R23: 100, Resistor_SMD:R_0603_1608Metric, F.Cu at (172.9, 100.0)
- added R24: 100, Resistor_SMD:R_0603_1608Metric, F.Cu at (135.4, 100.3)
- added R25: 100, Resistor_SMD:R_0603_1608Metric, F.Cu at (153.0, 101.1)
- added U2: STSPIN240, Package_DFN_QFN:VQFN-16-1EP_3x3mm_P0.5mm_EP1.8x1.8mm, F.Cu at (149.2, 106.6)
- added U3: LP5907MFX-1.2, Package_TO_SOT_SMD:SOT-23-5, F.Cu at (181.9, 90.2)
- added U4: HC-SR04, minimouse:HC-SR04, F.Cu at (150.0, 69.1)
- moved C5 23.9 mm to (147.1, 82.5), turned to 90 degrees
- moved C1 20.5 mm to (160.3, 81.5)
- moved C2 15.2 mm to (160.3, 83.2), turned to 180 degrees
- moved R9 4.42 mm to (148.1, 76.8)
- moved C6 4.07 mm to (142.8, 86.8), turned to 180 degrees
- moved C4 4.04 mm to (152.6, 96.4), turned to -90 degrees
- moved C3 3.97 mm to (142.9, 90.8)
- moved R8 3.29 mm to (153.7, 78.7)
- moved R1 3.22 mm to (151.7, 78.7)
- moved R2 3.03 mm to (141.1, 98.2)
- moved R6 2.13 mm to (149.0, 98.0)
- moved R7 2.11 mm to (150.5, 98.0)
- moved R4 1.51 mm to (145.4, 98.2)
- moved R5 1.51 mm to (146.9, 98.2)
- moved R3 1.26 mm to (142.8, 98.2)
Connections:
- R8 pad 1: /mcu/UART1_TX -> /external_uart/EXT_UART_RX
- U1 pad 43: /mcu/UART1_RX -> /external_uart/EXT_UART_TX
Routing:
- net /mcu/TIM15_CH1: track 0.00 -> 10.3 mm
- net /motor_control/TOFF: track 0.00 -> 8.94 mm
- net /mcu/IN_B2: track 0.00 -> 8.76 mm
- net /mcu/TIM15_CH2: track 0.00 -> 8.40 mm
- net /mcu/OUT_A4: track 0.00 -> 7.86 mm, vias 0 -> 2
- net Net-(U1-PA2): track 0.00 -> 7.03 mm
- net Net-(U1-PA3): track 0.00 -> 6.33 mm
- net Net-(U1-PA4): track 0.00 -> 5.09 mm
- net Net-(U1-PA5): track 0.00 -> 4.15 mm
- net Net-(U1-PB0): track 0.00 -> 3.73 mm
- net Net-(U1-PB1): track 0.00 -> 3.65 mm
- net +3.3V: track 0.00 -> 1.96 mm

Commit message: [Routage PCB]
Parts:
- moved R15 11.1 mm to (161.4, 101.8), turned to -90 degrees
- moved C15 8.79 mm to (138.7, 101.0), turned to 0 degrees
- moved R14 8.50 mm to (159.1, 101.8), turned to 90 degrees
- moved J3 4.12 mm to (127.7, 104.1)
- moved C13 3.55 mm to (125.7, 82.3)
- moved J4 3.55 mm to (121.8, 79.9)
- moved R20 3.55 mm to (125.8, 84.9), turned to 180 degrees
- moved R24 3.37 mm to (135.0, 97.0), turned to -90 degrees
- moved R22 3.30 mm to (132.9, 97.0), turned to -90 degrees
- moved C4 2.73 mm to (155.2, 95.8)
- moved R25 1.86 mm to (154.4, 100.0)
- moved C8 1.77 mm to (162.3, 99.5)
- moved R11 1.77 mm to (160.8, 97.7)
- moved R10 1.77 mm to (159.1, 99.5)
- moved R21 1.57 mm to (171.1, 98.6), turned to -90 degrees
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Routing:
- net +BATT: track 0.00 -> 87.7 mm
- net /motorB/MB: track 0.00 -> 36.2 mm
- net /motorA/MB: track 0.00 -> 32.6 mm
- net /mcu/SWO: track 0.00 -> 30.1 mm
- net /mcu/TIM3_CH1: track 0.00 -> 27.6 mm, vias 0 -> 4
- net GND: track 0.00 -> 26.9 mm, vias 0 -> 19
- net /mcu/SWDCLK: track 0.00 -> 26.1 mm
- net +3.3V: track 1.96 -> 27.2 mm
- net /mcu/SWDIO: track 0.00 -> 24.3 mm
- net /mcu/TIM3_CH2: track 0.00 -> 24.3 mm, vias 0 -> 1
- net /motorA/MA: track 0.00 -> 16.3 mm
- net /mcu/TIM2_CH1: track 0.00 -> 15.6 mm
- net /mcu/TIM2_CH2: track 0.00 -> 13.9 mm
- net /mcu/TIM8_CH2: track 0.00 -> 13.3 mm
- net Net-(U2-SENSEA): track 0.00 -> 13.2 mm
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
Commit message: Fin Tp minimouse
Parts:
- removed the U4 at (150.0, 69.1)
- added C7: 100n, Capacitor_SMD:C_0603_1608Metric, F.Cu at (170.9, 81.3)
- added D2: DZ2S030X0L, Diode_SMD:D_SOD-523, F.Cu at (160.2, 135.1)
- added Q1: NMOS, Package_TO_SOT_SMD:SOT-23, F.Cu at (157.3, 134.1)
- added R13: 10k, Resistor_SMD:R_0603_1608Metric, F.Cu at (171.0, 78.8)
- added R26: 10k, Resistor_SMD:R_0603_1608Metric, F.Cu at (161.9, 135.1)
- added SW1: SW_Push, Button_Switch_SMD:SW_Push_1P1T_NO_CK_KSC7xxJ, F.Cu at (177.8, 79.3)
- moved J4 41.4 mm to (161.7, 68.8)
- moved C13 41.0 mm to (165.2, 71.3)
- moved R20 30.3 mm to (155.3, 78.2), turned to 90 degrees
- moved D1 11.8 mm to (174.7, 90.8)
- moved R18 11.8 mm to (174.7, 94.0)
- moved C2 11.8 mm to (158.0, 94.8), turned to 0 degrees
- moved R1 11.6 mm to (158.1, 69.0)
- moved C12 8.68 mm to (177.3, 90.8), turned to -90 degrees
- moved C1 5.79 mm to (166.0, 82.5), turned to 90 degrees
- moved C11 5.65 mm to (182.7, 91.9), turned to 90 degrees
- moved BOOT0 4.19 mm to (156.1, 73.3)
- moved R8 4.00 mm to (157.6, 78.2)
- moved U3 2.43 mm to (179.8, 91.4), turned to 90 degrees
- moved R16 1.76 mm to (158.3, 113.7)
- moved J1 1.61 mm to (163.4, 85.2), turned to 180 degrees
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Connections:
- J5 pad 2: +BATT -> Net-(J5-Pin_2)
Routing:
- net +BATT: track 87.7 -> 244.4 mm, vias 0 -> 2
- net +3.3V: track 27.2 -> 72.5 mm
- net /mcu/~{RESET}: track 2.73 -> 32.9 mm, vias 0 -> 2
- net GND: track 26.9 -> 48.7 mm, vias 19 -> 27
- net /motorB/MA: track 1.85 -> 21.4 mm, vias 0 -> 2
- net /mcu/SWO: track 30.1 -> 12.1 mm
- net Net-(U2-SENSEB): track 0.00 -> 15.3 mm, vias 0 -> 2
- net /mcu/SWDIO: track 24.3 -> 9.20 mm
- net /mcu/SWDCLK: track 26.1 -> 11.5 mm
- net /mcu/BOOT0: track 6.93 -> 20.9 mm
- net Net-(C7-Pad2): track 0.00 -> 11.6 mm
- net Net-(J5-Pin_2): track 0.00 -> 9.95 mm
- net /external_uart/EXT_UART_TX: track 2.26 -> 9.65 mm
- net Net-(D2-A): track 0.00 -> 5.86 mm
- net Net-(J2-Pin_3): track 0.00 -> 4.66 mm
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- added copper zone on F.Cu, net +3.3V
- added copper zone on B.Cu, net GND
- added copper zone on F.Cu, net GND
