File: mm_mcu.kicad_sch (KiCad schematic)
At the start: 18 parts, among them J1 Conn_ARM_JTAG_SWD_10, U1 STM32F030C8Tx

Commit message: Fin Tp minimouse
Parts:
- added C7: 100n, Capacitor_SMD:C_0603_1608Metric, symbol minimouse:C
- added R13: 10k, Resistor_SMD:R_0603_1608Metric, symbol minimouse:R
- added SW1: SW_Push, Button_Switch_SMD:SW_Push_1P1T_NO_CK_KSC7xxJ, symbol Switch:SW_Push
Connections:
- net GND: now also C7.1, SW1.1
- net ~{RESET}: now also R13.2
- new net: C7.2, R13.1, SW1.2
Changed lines of the file:
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@@
   (junction (at 140.97 123.19) (diameter 0) (color 0 0 0 0)
   )
+  (junction (at 97.79 38.1) (diameter 0) (color 0 0 0 0)
+  )
   (junction (at 142.24 35.56) (diameter 0) (color 0 0 0 0)
   )
@@
   )
   (junction (at 220.98 27.94) (diameter 0) (color 0 0 0 0)
+  )
+  (junction (at 78.74 36.83) (diameter 0) (color 0 0 0 0)
   )
   (junction (at 48.26 182.88) (diameter 0) (color 0 0 0 0)
@@
     (stroke (width 0) (type default))
   )
+  (wire (pts (xy 97.79 38.1) (xy 97.79 31.75))
+    (stroke (width 0) (type default))
+  )
   (wire (pts (xy 220.98 38.1) (xy 220.98 39.37))
     (stroke (width 0) (type default))
@@
     (stroke (width 0) (type default))
   )
+  (wire (pts (xy 78.74 31.75) (xy 83.82 31.75))
+    (stroke (width 0) (type default))
+  )
   (wire (pts (xy 48.26 182.88) (xy 48.26 185.42))
     (stroke (width 0) (type default))
@@
     (stroke (width 0) (type default))
   )
+  (wire (pts (xy 78.74 38.1) (xy 78.74 36.83))
+    (stroke (width 0) (type default))
+  )
   (wire (pts (xy 238.76 27.94) (xy 238.76 30.48))
     (stroke (width 0) (type default))
@@
     (stroke (width 0) (type default))
   )
+  (wire (pts (xy 92.71 38.1) (xy 97.79 38.1))
+    (stroke (width 0) (type default))
+  )
   (wire (pts (xy 139.7 35.56) (xy 139.7 36.83))
     (stroke (width 0) (type default))
@@
     (stroke (width 0) (type default))
   )
+  (wire (pts (xy 85.09 38.1) (xy 78.74 38.1))
+    (stroke (width 0) (type default))
+  )
+  (wire (pts (xy 97.79 41.91) (xy 97.79 38.1))
+    (stroke (width 0) (type default))
+  )
   (wire (pts (xy 144.78 36.83) (xy 144.78 35.56))
     (stroke (width 0) (type default))
@@
     (stroke (width 0) (type default))
   )
+  (wire (pts (xy 71.12 36.83) (xy 78.74 36.83))
+    (stroke (width 0) (type default))
+  )
   (wire (pts (xy 238.76 38.1) (xy 238.76 39.37))
     (stroke (width 0) (type default))
@@
     (stroke (width 0) (type default))
   )
-  (wire (pts (xy 109.22 41.91) (xy 124.46 41.91))
+  (wire (pts (xy 105.41 41.91) (xy 124.46 41.91))
+    (stroke (width 0) (type default))
+  )
+  (wire (pts (xy 78.74 36.83) (xy 78.74 31.75))
     (stroke (width 0) (type default))
   )
   (wire (pts (xy 154.94 44.45) (xy 182.88 44.45))
+    (stroke (width 0) (type default))
+  )
+  (wire (pts (xy 97.79 31.75) (xy 93.98 31.75))
     (stroke (width 0) (type default))
   )
@@
         (path "/d8fa4cba-2469-4231-847f-065b6b829f44/b5d7e952-00af-4b6f-924a-ee43c62726d2"
           (reference "J1") (unit 1)
+        )
+      )
+    )
+  )
+  (symbol (lib_id "minimouse:C") (at 88.9 38.1 90) (unit 1)
+    (in_bom yes) (on_board yes) (dnp no) (fields_autoplaced)
+    (property "Reference" "C7" (at 88.9 30.48 90)
+      (effects (font (size 1.27 1.27)))
+    )
+    (property "Value" "100n" (at 88.9 33.02 90)
+      (effects (font (size 1.27 1.27)))
+    )
+    (property "Footprint" "Capacitor_SMD:C_0603_1608Metric" (at 92.71 37.1348 0)
+      (effects (font (size 1.27 1.27)) hide)
+    )
+    (property "Datasheet" "~" (at 88.9 38.1 0)
+      (effects (font (size 1.27 1.27)) hide)
+    )
+    (pin "1")
+    (pin "2")
+    (instances
+      (project "minimouse"
+        (path "/d8fa4cba-2469-4231-847f-065b6b829f44/b5d7e952-00af-4b6f-924a-ee43c62726d2"
+          (reference "C7") (unit 1)
         )
       )
@@
     )
   )
+  (symbol (lib_id "power:GND") (at 71.12 36.83 0) (unit 1)
+    (in_bom yes) (on_board yes) (dnp no) (fields_autoplaced)
+    (property "Reference" "#PWR010" (at 71.12 43.18 0)
+      (effects (font (size 1.27 1.27)) hide)
+    )
+    (property "Value" "GND" (at 71.12 41.91 0)
+      (effects (font (size 1.27 1.27)))
+    )
+    (property "Footprint" "" (at 71.12 36.83 0)
+      (effects (font (size 1.27 1.27)) hide)
+    )
+    (property "Datasheet" "" (at 71.12 36.83 0)
+      (effects (font (size 1.27 1.27)) hide)
+    )
+    (pin "1")
+    (instances
+      (project "minimouse"
+        (path "/d8fa4cba-2469-4231-847f-065b6b829f44/b5d7e952-00af-4b6f-924a-ee43c62726d2"
+          (reference "#PWR010") (unit 1)
+        )
+      )
+    )
+  )
   (symbol (lib_id "Device:R") (at 166.37 49.53 90) (unit 1)
     (in_bom yes) (on_board yes) (dnp no)
@@
     )
   )
+  (symbol (lib_id "Switch:SW_Push") (at 88.9 31.75 0) (unit 1)
+    (in_bom yes) (on_board yes) (dnp no) (fields_autoplaced)
+    (property "Reference" "SW1" (at 88.9 24.13 0)
+      (effects (font (size 1.27 1.27)))
+    )
+    (property "Value" "SW_Push" (at 88.9 26.67 0)
+      (effects (font (size 1.27 1.27)))
+    )
+    (property "Footprint" "Button_Switch_SMD:SW_Push_1P1T_NO_CK_KSC7xxJ" (at 88.9 26.67 0)
+      (effects (font (size 1.27 1.27)) hide)
+    )
+    (property "Datasheet" "~" (at 88.9 26.67 0)
+      (effects (font (size 1.27 1.27)) hide)
+    )
+    (pin "1")
+    (pin "2")
+    (instances
+      (project "minimouse"
+        (path "/d8fa4cba-2469-4231-847f-065b6b829f44/b5d7e952-00af-4b6f-924a-ee43c62726d2"
+          (reference "SW1") (unit 1)
+        )
+      )
+    )
+  )
   (symbol (lib_id "Device:C") (at 238.76 34.29 0) (unit 1)
     (in_bom yes) (on_board yes) (dnp no)
@@
         )
       )
+    )
+  )
+  (symbol (lib_id "minimouse:R") (at 101.6 41.91 90) (unit 1)
+    (in_bom yes) (on_board yes) (dnp no) (fields_autoplaced)
+    (property "Reference" "R13" (at 101.6 35.56 90)
+      (effects (font (size 1.27 1.27)))
+    )
+    (property "Value" "10k" (at 101.6 38.1 90)
+      (effects (font (size 1.27 1.27)))
+    )
+    (property "Footprint" "Resistor_SMD:R_0603_1608Metric" (at 101.6 43.688 90)
+      (effects (font (size 1.27 1.27)) hide)
+    )
+    (property "Datasheet" "~" (at 101.6 41.91 0)
+      (effects (font (size 1.27 1.27)) hide)
+    )
+    (pin "1")
+    (pin "2")
+    (instances
+      (project "minimouse"
+        (path "/d8fa4cba-2469-4231-847f-065b6b829f44/b5d7e952-00af-4b6f-924a-ee43c62726d2"
+          (reference "R13") (unit 1)
+        )
+      )
