File: mm_power.kicad_sch (KiCad schematic)
At the start: 1 part, among them J5 Conn_01x02

Commit message: fin tp2
Parts:
- added C11: 1uF, Capacitor_SMD:C_0603_1608Metric, symbol minimouse:C
- added C12: 1uF, symbol minimouse:C
- added D1: LED, LED_SMD:LED_0603_1608Metric, symbol Device:LED
- added R18: 600, Resistor_SMD:R_0603_1608Metric, symbol minimouse:R
- added U3: LP5907MFX-1.2, Package_TO_SOT_SMD:SOT-23-5, symbol Regulator_Linear:LP5907MFX-1.2
Connections:
- net +BATT: now also C11.1, U3.1 (IN), U3.3 (EN)
- net GND: now also C11.2, C12.2, R18.2, U3.2 (GND)
- new net: D1.1 (K), R18.1
- new net +3.3V: C12.1, D1.2 (A), U3.5 (OUT)

Commit message: [Debut du routage TP3]
Parts:
- C11: value 1uF -> 2.2uF
- C12: value 1uF -> 2.2uF; footprint (none) -> Capacitor_SMD:C_0603_1608Metric
- R18: value 600 -> 330
Changed lines of the file:
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@@
       (effects (font (size 1.27 1.27)) (justify left))
     )
-    (property "Value" "1uF" (at 165.1 88.9 0)
+    (property "Value" "2.2uF" (at 165.1 88.9 0)
       (effects (font (size 1.27 1.27)) (justify left))
     )
-    (property "Footprint" "" (at 162.2552 91.44 0)
+    (property "Footprint" "Capacitor_SMD:C_0603_1608Metric" (at 162.2552 91.44 0)
       (effects (font (size 1.27 1.27)) hide)
     )
@@
       (effects (font (size 1.27 1.27)) (justify left))
     )
-    (property "Value" "600" (at 196.85 100.33 0)
+    (property "Value" "330" (at 196.85 100.33 0)
       (effects (font (size 1.27 1.27)) (justify left))
     )
@@
       (effects (font (size 1.27 1.27)) (justify left))
     )
-    (property "Value" "1uF" (at 135.89 88.9 0)
+    (property "Value" "2.2uF" (at 135.89 88.9 0)
       (effects (font (size 1.27 1.27)) (justify left))
     )

Commit message: [Routage PCB]
Changed lines of the file:
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@@
   (junction (at 86.36 95.25) (diameter 0) (color 0 0 0 0)
   )
+  (junction (at 167.64 82.55) (diameter 0) (color 0 0 0 0)
+  )
   (junction (at 161.29 82.55) (diameter 0) (color 0 0 0 0)
   )
@@
     (stroke (width 0) (type default))
   )
-  (wire (pts (xy 194.31 73.66) (xy 194.31 82.55))
+  (wire (pts (xy 167.64 82.55) (xy 194.31 82.55))
     (stroke (width 0) (type default))
   )
@@
         )
       )
-    )
-  )
-  (symbol (lib_id "power:+3.3V") (at 194.31 73.66 0) (unit 1)
-    (in_bom yes) (on_board yes) (dnp no) (fields_autoplaced)
-    (property "Reference" "#PWR030" (at 194.31 77.47 0)
-      (effects (font (size 1.27 1.27)) hide)
-    )
-    (property "Value" "+3.3V" (at 194.31 68.58 0)
-      (effects (font (size 1.27 1.27)))
-    )
-    (property "Footprint" "" (at 194.31 73.66 0)
-      (effects (font (size 1.27 1.27)) hide)
-    )
-    (property "Datasheet" "" (at 194.31 73.66 0)
-      (effects (font (size 1.27 1.27)) hide)
-    )
-    (pin "1")
-    (instances
-      (project "minimouse"
-        (path "/d8fa4cba-2469-4231-847f-065b6b829f44/3f9b0845-5778-418c-a7a8-03da2392145e"
-          (reference "#PWR030") (unit 1)
-        )
-      )

Commit message: Fin Tp minimouse
Parts:
- added D2: DZ2S030X0L, Diode_SMD:D_SOD-523, symbol Diode:DZ2S030X0L
- added Q1: NMOS, Package_TO_SOT_SMD:SOT-23, symbol Simulation_SPICE:NMOS
- added R26: 10k, Resistor_SMD:R_0603_1608Metric, symbol minimouse:R
Connections:
- net +BATT: now also D2.1 (K), Q1.3 (S); no longer J5.2 (Pin_2)
- net GND: now also R26.2
- new net: D2.2 (A), Q1.2 (G), R26.1
- new net: J5.2 (Pin_2), Q1.1 (D)
Changed lines of the file:
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@@
   (junction (at 138.43 82.55) (diameter 0) (color 0 0 0 0)
   )
-  (junction (at 86.36 82.55) (diameter 0) (color 0 0 0 0)
+  (junction (at 113.03 87.63) (diameter 0) (color 0 0 0 0)
+  )
+  (junction (at 116.84 77.47) (diameter 0) (color 0 0 0 0)
   )
   (junction (at 86.36 95.25) (diameter 0) (color 0 0 0 0)
   )
+  (junction (at 127 77.47) (diameter 0) (color 0 0 0 0)
+  )
   (junction (at 167.64 82.55) (diameter 0) (color 0 0 0 0)
   )
+  (junction (at 90.17 82.55) (diameter 0) (color 0 0 0 0)
+  )
   (junction (at 161.29 82.55) (diameter 0) (color 0 0 0 0)
   )
@@
     (stroke (width 0) (type default))
   )
+  (wire (pts (xy 109.22 87.63) (xy 113.03 87.63))
+    (stroke (width 0) (type default))
+  )
   (wire (pts (xy 167.64 82.55) (xy 167.64 74.93))
     (stroke (width 0) (type default))
   )
+  (wire (pts (xy 114.3 77.47) (xy 116.84 77.47))
+    (stroke (width 0) (type default))
+  )
   (wire (pts (xy 140.97 82.55) (xy 138.43 82.55))
     (stroke (width 0) (type default))
@@
     (stroke (width 0) (type default))
   )
-  (wire (pts (xy 95.25 82.55) (xy 86.36 82.55))
-    (stroke (width 0) (type default))
-  )
-  (wire (pts (xy 86.36 74.93) (xy 86.36 82.55))
+  (wire (pts (xy 95.25 82.55) (xy 90.17 82.55))
     (stroke (width 0) (type default))
   )
@@
     (stroke (width 0) (type default))
   )
+  (wire (pts (xy 113.03 87.63) (xy 113.03 92.71))
+    (stroke (width 0) (type default))
+  )
   (wire (pts (xy 95.25 92.71) (xy 95.25 95.25))
     (stroke (width 0) (type default))
@@
     (stroke (width 0) (type default))
   )
+  (wire (pts (xy 109.22 85.09) (xy 109.22 87.63))
+    (stroke (width 0) (type default))
+  )
+  (wire (pts (xy 116.84 77.47) (xy 116.84 80.01))
+    (stroke (width 0) (type default))
+  )
+  (wire (pts (xy 113.03 87.63) (xy 116.84 87.63))
+    (stroke (width 0) (type default))
+  )
   (wire (pts (xy 80.01 87.63) (xy 86.36 87.63))
     (stroke (width 0) (type default))
@@
     (stroke (width 0) (type default))
   )
+  (wire (pts (xy 90.17 77.47) (xy 90.17 82.55))
+    (stroke (width 0) (type default))
+  )
   (wire (pts (xy 132.08 82.55) (xy 132.08 83.82))
     (stroke (width 0) (type default))
@@
     (stroke (width 0) (type default))
   )
+  (wire (pts (xy 104.14 77.47) (xy 90.17 77.47))
+    (stroke (width 0) (type default))
+  )
   (wire (pts (xy 161.29 82.55) (xy 167.64 82.55))
     (stroke (width 0) (type default))
@@
     (stroke (width 0) (type default))
   )
-  (wire (pts (xy 127 82.55) (xy 127 73.66))
+  (wire (pts (xy 127 82.55) (xy 127 77.47))
+    (stroke (width 0) (type default))
+  )
+  (wire (pts (xy 113.03 100.33) (xy 113.03 101.6))
     (stroke (width 0) (type default))
   )
@@
     (stroke (width 0) (type default))
   )
+  (wire (pts (xy 116.84 77.47) (xy 127 77.47))
+    (stroke (width 0) (type default))
+  )
   (wire (pts (xy 140.97 85.09) (xy 138.43 85.09))
     (stroke (width 0) (type default))
@@
     (stroke (width 0) (type default))
   )
+  (wire (pts (xy 127 77.47) (xy 127 73.66))
+    (stroke (width 0) (type default))
+  )
+  (wire (pts (xy 90.17 82.55) (xy 86.36 82.55))
+    (stroke (width 0) (type default))
+  )
   (wire (pts (xy 80.01 90.17) (xy 86.36 90.17))
     (stroke (width 0) (type default))
-  )
-  (symbol (lib_id "power:+BATT") (at 86.36 74.93 0) (unit 1)
-    (in_bom yes) (on_board yes) (dnp no) (fields_autoplaced)
-    (property "Reference" "#PWR036" (at 86.36 78.74 0)
-      (effects (font (size 1.27 1.27)) hide)
-    )
-    (property "Value" "+BATT" (at 86.36 69.85 0)
-      (effects (font (size 1.27 1.27)))
-    )
-    (property "Footprint" "" (at 86.36 74.93 0)
-      (effects (font (size 1.27 1.27)) hide)
-    )
-    (property "Datasheet" "" (at 86.36 74.93 0)
-      (effects (font (size 1.27 1.27)) hide)
-    )
-    (pin "1")
-    (instances
-      (project "minimouse"
-        (path "/d8fa4cba-2469-4231-847f-065b6b829f44/3f9b0845-5778-418c-a7a8-03da2392145e"
-          (reference "#PWR036") (unit 1)
-        )
-      )
-    )
   )
   (symbol (lib_id "power:GND") (at 194.31 109.22 0) (unit 1)
@@
     )
   )
+  (symbol (lib_id "Diode:DZ2S030X0L") (at 116.84 83.82 270) (unit 1)
+    (in_bom yes) (on_board yes) (dnp no) (fields_autoplaced)
+    (property "Reference" "D2" (at 119.38 82.55 90)
+      (effects (font (size 1.27 1.27)) (justify left))
+    )
+    (property "Value" "DZ2S030X0L" (at 119.38 85.09 90)
+      (effects (font (size 1.27 1.27)) (justify left))
+    )
+    (property "Footprint" "Diode_SMD:D_SOD-523" (at 112.395 83.82 0)
+      (effects (font (size 1.27 1.27)) hide)
+    )
+    (property "Datasheet" "https://industrial.panasonic.com/content/data/SC/ds/ds4/DZ2S03000L_E.pdf" (at 116.84 83.82 0)
+      (effects (font (size 1.27 1.27)) hide)
+    )
+    (pin "2")
+    (pin "1")
+    (instances
+      (project "minimouse"
+        (path "/d8fa4cba-2469-4231-847f-065b6b829f44/3f9b0845-5778-418c-a7a8-03da2392145e"
+          (reference "D2") (unit 1)
+        )
+      )
+    )
+  )
   (symbol (lib_id "Device:LED") (at 194.31 86.36 90) (unit 1)
     (in_bom yes) (on_board yes) (dnp no) (fields_autoplaced)
@@
         (path "/d8fa4cba-2469-4231-847f-065b6b829f44/3f9b0845-5778-418c-a7a8-03da2392145e"
           (reference "D1") (unit 1)
+        )
+      )
+    )
+  )
+  (symbol (lib_id "power:GND") (at 113.03 101.6 0) (unit 1)
+    (in_bom yes) (on_board yes) (dnp no) (fields_autoplaced)
+    (property "Reference" "#PWR012" (at 113.03 107.95 0)
+      (effects (font (size 1.27 1.27)) hide)
+    )
+    (property "Value" "GND" (at 113.03 106.68 0)
+      (effects (font (size 1.27 1.27)))
+    )
+    (property "Footprint" "" (at 113.03 101.6 0)
+      (effects (font (size 1.27 1.27)) hide)
+    )
+    (property "Datasheet" "" (at 113.03 101.6 0)
+      (effects (font (size 1.27 1.27)) hide)
+    )
+    (pin "1")
+    (instances
+      (project "minimouse"
+        (path "/d8fa4cba-2469-4231-847f-065b6b829f44/3f9b0845-5778-418c-a7a8-03da2392145e"
+          (reference "#PWR012") (unit 1)
         )
       )
@@
         )
       )
+    )
+  )
+  (symbol (lib_id "Simulation_SPICE:NMOS") (at 109.22 80.01 90) (unit 1)
+    (in_bom yes) (on_board yes) (dnp no) (fields_autoplaced)
+    (property "Reference" "Q1" (at 109.22 71.12 90)
+      (effects (font (size 1.27 1.27)))
+    )
+    (property "Value" "NMOS" (at 109.22 73.66 90)
+      (effects (font (size 1.27 1.27)))
+    )
+    (property "Footprint" "Package_TO_SOT_SMD:SOT-23" (at 106.68 74.93 0)
+      (effects (font (size 1.27 1.27)) hide)
+    )
+    (property "Datasheet" "https://ngspice.sourceforge.io/docs/ngspice-manual.pdf" (at 121.92 80.01 0)
+      (effects (font (size 1.27 1.27)) hide)
+    )
+    (property "Sim.Device" "NMOS" (at 126.365 80.01 0)
+      (effects (font (size 1.27 1.27)) hide)
+    )
+    (property "Sim.Type" "VDMOS" (at 128.27 80.01 0)
+      (effects (font (size 1.27 1.27)) hide)
+    )
+    (property "Sim.Pins" "1=D 2=G 3=S" (at 124.46 80.01 0)
+      (effects (font (size 1.27 1.27)) hide)
+    )
+    (pin "2")
+    (pin "1")
+    (pin "3")
+    (instances
+      (project "minimouse"
+        (path "/d8fa4cba-2469-4231-847f-065b6b829f44/3f9b0845-5778-418c-a7a8-03da2392145e"
+          (reference "Q1") (unit 1)
+        )
+      )
+    )
+  )
+  (symbol (lib_id "minimouse:R") (at 113.03 96.52 0) (unit 1)
+    (in_bom yes) (on_board yes) (dnp no) (fields_autoplaced)
+    (property "Reference" "R26" (at 115.57 95.25 0)
+      (effects (font (size 1.27 1.27)) (justify left))
+    )
+    (property "Value" "10k" (at 115.57 97.79 0)
+      (effects (font (size 1.27 1.27)) (justify left))
+    )
+    (property "Footprint" "Resistor_SMD:R_0603_1608Metric" (at 111.252 96.52 90)
+      (effects (font (size 1.27 1.27)) hide)
+    )
+    (property "Datasheet" "~" (at 113.03 96.52 0)
+      (effects (font (size 1.27 1.27)) hide)
+    )
+    (pin "2")
+    (pin "1")
+    (instances
+      (project "minimouse"
+        (path "/d8fa4cba-2469-4231-847f-065b6b829f44/3f9b0845-5778-418c-a7a8-03da2392145e"
+          (reference "R26") (unit 1)
+        )
+      )
